File: pro_event_light_a_mkI/pro_event_light_a_mkI_modules.sch (EAGLE design)
At the start: 53 parts, among them K1 62201021121

Commit message: commit prior of trying to clone some parts
Parts:
- removed C1, C29, C34, C35: 1uF, Eagle_Wurth_Elektronik_Passive_Capacitors_rev15a:WCAP-CSGP_1206
- removed C10: 10uF, Eagle_Wurth_Elektronik_Passive_Capacitors_rev15a:WCAP-ASNP_4X5.5(DXL)
- removed C2: 220pF, Eagle_Wurth_Elektronik_Passive_Capacitors_rev15a:WCAP-CSGP_0603-WAVE
- removed C3: 45uF, Eagle_Wurth_Elektronik_Passive_Capacitors_rev15a:WCAP-ASNP_4X5.5(DXL)
- removed C4, C6, C7: 4.7uF, Eagle_Wurth_Elektronik_Passive_Capacitors_rev15a:WCAP-CSGP_0603-WAVE
- removed C5: 100nF, Eagle_Wurth_Elektronik_Passive_Capacitors_rev15a:WCAP-CSGP_0603-REFLOW
- removed D1, D2: MBR0540T1, mod_eagle_library_discrete_elements:MBR0540T1
- removed D3: 1N4148WS, mod_eagle_library_discrete_elements:1N4148WS
- removed K1: 62201021121, Board_to_Board_Connectors_rev15d:62201021121
- removed L1: 1uH, EagleLibrary_Wuerth_Elektronik_eiSos_rev16a:WE-LQ_1210
- removed MCU1: STM32L452RET6, mod_eagle_library_MCU_CPU:STM32L452RET6
- removed R10, R3, R7, R8, R9: 0R0, rcl:R-EU_R0603
- removed R11: 10K, rcl:R-EU_R0603
- removed R12: 17K5, rcl:R-EU_R0603
- removed R13: 27K, rcl:R-EU_R0603
- removed R2: (no value), rcl:R-EU_R0603
- removed R35, R36: 0R, rcl:R-EU_R0603
- removed U$10, U$11, U$15, U$8: (no value), mod-eagle_library_standard_passive_parts:PCB_MOUNTING_HOLES_M3
- removed U$4, U$5: LT1936, mod_eagle_library_pmic:LT1936
- removed U$7: ALPS_EC11D, mod_eagle_library_switches:ALPS_EC11D
- added C8/1, C8/2, C8/3, C8/4: (no value), Eagle_Wurth_Elektronik_Passive_Capacitors_rev15a:WCAP-CSGP_0603-WAVE
- added DZ1/1, DZ1/2, DZ1/3, DZ1/4: MBR0540T1, mod_eagle_library_discrete_elements:MBR0540T1
- added IC1/1, IC1/2, IC1/3, IC1/4: ILD4001, infineon:ILD4001
- added L2/1, L2/2, L2/3, L2/4: 68uH, EagleLibrary_Wuerth_Elektronik_eiSos_rev16a:WE-LQ_1210
- added R14/1, R14/2, R14/3, R14/4: (no value), rcl:R-EU_R0603
- added U1/1, U1/2, U1/3, U1/4: PMXB56EN, mod_eagle_library_discrete_elements:PMXB56EN
Connections:
- removed net N$15: C34.1, U$10.1
- removed net N$17: C35.1, U$15.1
- removed net N$18: C1.1, U$8.1
- removed net N$19: C5.2, MCU1G$2.VBAT, R3.1
- removed net N$20: MCU1G$2.PC14/OCS32_IN, R10.1
- removed net N$21: R8.1
- removed net N$26: MCU1G$2.PHO/OSC_IN, R9.1
- removed net N$27: MCU1G$2.PH1/OSC_OUT, R7.1
- removed net N$28: U$4.COMP, U$4.VC
- removed net N$30: C7.1, R13.1, U$4.SHDN
- removed net N$33: C2.1, D3.C, U$4.BOOST
- removed net N$34: C2.2, D1.C, L1.1, U$4.SW
- removed net N$35: R11.2, R12.2, U$4.FB
- removed net N$9: C29.1, U$11.1
- removed net NRESET: K1.6
- removed net S3V3_MCU_VDD: MCU1G$2.VDD_19, MCU1G$2.VDD_32, MCU1G$2.VDD_64, R2.1, R3.2
- removed net SUPPLY_3V3: C3.2, C4.1, D3.A, L1.2, R12.1
- removed net SWCLK: K1.9, MCU1G$1.PA14
- removed net SWDIO: K1.10, MCU1G$1.PA13
- removed net SWO: K1.8, R35.1
- removed net TDI: K1.7, R36.1
- removed net VIN: D2.A
- removed net VTREF: K1.1, R2.2
- new net DRIVER_LEDB/1: L2/2.1
- new net DRIVER_LEDG/1: L2/1.1
- new net DRIVER_LEDR/1: L2/3.1
- new net DRIVER_LEDW/1: L2/4.1
- new net ENABLE_LEDB/1: IC1/2.EN/PWM
- new net ENABLE_LEDG/1: IC1/1.EN/PWM
- new net ENABLE_LEDR/1: IC1/3.EN/PWM
- new net ENABLE_LEDW/1: IC1/4.EN/PWM
- new net N$1: DZ1/2.A, L2/2.2, U1/2.D
- new net N$2: IC1/1.VDRIVE, R14/1.2, U1/1.G
- new net N$29: DZ1/1.A, L2/1.2, U1/1.D
- new net N$32: DZ1/3.A, L2/3.2, U1/3.D
- new net N$36: IC1/3.VDRIVE, R14/3.2, U1/3.G
- new net N$37: DZ1/4.A, L2/4.2, U1/4.D
- new net N$38: IC1/4.VDRIVE, R14/4.2, U1/4.G
- new net N$8: IC1/2.VDRIVE, R14/2.2, U1/2.G
- new net VSENSE_LEDB/1: IC1/2.VSENSE
- new net VSENSE_LEDG/1: IC1/1.VSENSE
- new net VSENSE_LEDR/1: IC1/3.VSENSE
- new net VSENSE_LEDW/1: IC1/4.VSENSE
- net GND_MCU: now also C8/1.1, C8/2.1, C8/3.1, C8/4.1, IC1/1.GND, IC1/2.GND, IC1/3.GND, IC1/4.GND, R14/1.1, R14/2.1, R14/3.1, R14/4.1, U1/1.S, U1/2.S, U1/3.S, U1/4.S; no longer C1.2, C10.1, C29.2, C3.1, C34.2, C35.2, C4.2, C5.1, C6.2, C7.2, D1.A, K1.2, K1.3, MCU1G$2.VSS_18, MCU1G$2.VSS_47, MCU1G$2.VSS_63, R10.2, R11.1, R35.2, R36.2, R7.2, R8.2, R9.2, U$4.GND1, U$4.GND2
- net SUPPLY_24V: now also C8/1.2, C8/2.2, C8/3.2, C8/4.2, DZ1/1.C, DZ1/2.C, DZ1/3.C, DZ1/4.C, IC1/1.VS, IC1/2.VS, IC1/3.VS, IC1/4.VS; no longer C10.2, C6.1, D2.C, R13.2, U$4.VIN
Other:
- note removed: "12V"
- note removed: "3V3"
- note removed: "Attention: This Symbol is mirrored compared to the package-> mirror it in the layout if necessary"
- note removed: "C_out = 150/V_out C_out = 45uF"
- note removed: "L=2.2(V_out + V_D) L=8.36uH~=10uH"
- note removed: "V_out = 1.200V * (1 + R_1 / R_2)"
- note removed: "V_out = 12V (3.3V/ 1.200V - 1) * R_2 = R_1 R_2 = 10k R_1 = 90k"
- note removed: "V_out = 3.3V (3.3V/ 1.200V - 1) * R_2 = R_1 R_2 = 10k R_1 = 17.5k"
- note removed: "boost voltage generation C=0.22uF fast switching diode 1N4148 or 1N914"
- note removed: "take a small capacitor and a larger maybe electrolytic one 4.7uF"
