File: pro_event_light_a_mkI/pro_event_light_a_mkI_base_board.brd (EAGLE design)
At the start: 39.6 x 59.4 mm, 59 parts, among them IC1 ILD4001, IC2 ILD4001, IC3 ILD4001, IC4 ILD4001, K1 62201021121

Commit message: commit prior of trying to clone some parts
Parts:
- removed IC1, IC2, IC3, IC4: ILD4001, infineon:SC74_INFINEON
- removed U$1, U$2, U$3, U$6: PMXB56EN, mod_eagle_library_discrete_elements:DFN1010D-3
- removed U$5: LT1936, mod_eagle_library_pmic:MSOP8
- added C10: 10uF, Eagle_Wurth_Elektronik_Passive_Capacitors_rev15a:2.6X1.6X1(BXCXA)
- added C8/1: (no value), Eagle_Wurth_Elektronik_Passive_Capacitors_rev15a:WCAP-CSGP_0603_WAVE
- added DZ1/1: MBR0540T1, mod_eagle_library_discrete_elements:SOD123
- added IC1/1: ILD4001, infineon:SC74_INFINEON
- added L2/1: 68uH, EagleLibrary_Wuerth_Elektronik_eiSos_rev16a:WE-LQ_M
- added R13: 27K, rcl:R0603
- added R14/1: (no value), rcl:R0603
- added U1/1: PMXB56EN, mod_eagle_library_discrete_elements:DFN1010D-3
- C2: value (none) -> 220pF; device rcl:C0603 -> Eagle_Wurth_Elektronik_Passive_Capacitors_rev15a:WCAP-CSGP_0603_WAVE
- C3: value (none) -> 45uF; device rcl:C0603 -> Eagle_Wurth_Elektronik_Passive_Capacitors_rev15a:2.6X1.6X1(BXCXA)
- C4, C6, C7: value (none) -> 4.7uF; device rcl:C0603 -> Eagle_Wurth_Elektronik_Passive_Capacitors_rev15a:WCAP-CSGP_0603_WAVE
- D1, D2: value BAS40 -> MBR0540T1; device diode:SOT23 -> mod_eagle_library_discrete_elements:SOD123
- D3: value GF1 -> 1N4148WS; device diode:SMA-DO214AC -> mod_eagle_library_discrete_elements:SOD323
- L1: value MSS7341 -> 1uH; device inductor-coilcraft:MSS7341 -> EagleLibrary_Wuerth_Elektronik_eiSos_rev16a:WE-LQ_M
- R11: value (none) -> 10K
- R12: value (none) -> 17K5
- moved R6 135.5 mm to (31.8, -93.2), turned to 0 degrees
- moved R5 135.4 mm to (27.9, -93.2), turned to 0 degrees
- moved R4 135.3 mm to (24.1, -93.2), turned to 0 degrees
- moved R1 135.2 mm to (20.3, -93.2), turned to 0 degrees
- moved LEDR5 117.4 mm to (6.86, -84.3), turned to 0 degrees
- moved LEDR6 104.4 mm to (30.5, -84.3), turned to 0 degrees
- moved LEDR4 104.2 mm to (-16.8, -84.3), turned to 0 degrees
- moved LEDR1 103.8 mm to (-16.8, -68.8), turned to 0 degrees
- moved C7 95.0 mm to (16.8, 50.0)
- moved C6 89.4 mm to (17.8, 46.7)
- moved LEDR2 89.1 mm to (6.86, -68.8), turned to 0 degrees
- moved LEDB4 85.7 mm to (-16.8, -53.3), turned to 0 degrees
- moved LEDR3 80.3 mm to (30.5, -68.8), turned to 0 degrees
- moved LEDB1 67.3 mm to (-16.8, -37.8), turned to 0 degrees
- moved LEDB3 63.7 mm to (30.5, -37.8), turned to 0 degrees
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Connections:
- net N$16 renamed VSENSE_LEDR
- net N$2 renamed VSENSE_LEDG
- net N$23 renamed VSENSE_LEDW
- net N$5 renamed VSENSE_LEDB
- removed net GND: IC1.2, IC1.5, IC2.2, IC2.5, IC3.2, IC3.5, IC4.2, IC4.5
- removed net N$1: U$1.2, U$2.2, U$3.2
- removed net N$10: R5.2
- removed net N$11: R6.2
- removed net N$13: R4.2
- removed net N$22: LEDR2.3, LEDR2.4, LEDR4.3, LEDR4.4, LEDR6.3, LEDR6.4, U$2.3
- removed net N$24: LEDW2.3, LEDW2.4, U$6.3
- removed net N$31: LEDB2.3, LEDB2.4, LEDB4.3, LEDB4.4, U$3.3
- removed net N$36: C4.1, C7.1, D3.A, L1.1, R12.1
- removed net N$8: R1.2
- new net DRIVER_LEDB: LEDB2.3, LEDB2.4, LEDB4.3, LEDB4.4
- new net DRIVER_LEDG: LEDG1.3, LEDG1.4
- new net DRIVER_LEDG/1: L2/1.1
- new net DRIVER_LEDR: LEDR2.3, LEDR2.4, LEDR4.3, LEDR4.4, LEDR6.3, LEDR6.4
- new net DRIVER_LEDW: LEDW2.3, LEDW2.4
- new net ENABLE_LEDG/1: IC1/1.3
- new net N$2: IC1/1.4, R14/1.2, U1/1.1
- new net SUPPLY_24V: C10.2, C6.1, C8/1.2, D2.C, DZ1/1.C, IC1/1.1, R1.2, R13.2, R4.2, R5.2, R6.2, U$4.2
- new net SUPPLY_3V3: C3.2, C4.1, D3.A, L1.2, R12.1
- new net VIN: D2.A
- new net VSENSE_LEDG/1: IC1/1.6
- net GND_MCU: now also C10.1, C3.1, C8/1.1, D1.A, IC1/1.2, IC1/1.5, R14/1.1, U1/1.2; no longer C3.2, D1.1
- net N$28: now also U$4.8
- net N$29: now also DZ1/1.A, L2/1.2, U1/1.3; no longer LEDG1.3, LEDG1.4, U$1.3
- net N$30: now also C7.1, R13.1, U$4.5; no longer C3.1, C6.1, U$4.2
- net N$33: now also D3.C; no longer D3.K
- net N$34: now also D1.C, L1.1; no longer D1.3, L1.2
Routing:
- net GND_MCU: track 207.9 -> 0.00 mm, vias 5 -> 0
- net VSENSE_LEDB: track 62.2 -> 0.00 mm
- net VSENSE_LEDR: track 59.7 -> 0.00 mm, vias 2 -> 0
- net N$22: track 59.0 -> 0.00 mm, vias 2 -> 0
- net N$31: track 57.4 -> 0.00 mm, vias 1 -> 0
- net S3V3_MCU_VDD: track 52.3 -> 0.00 mm
- net N$12: track 30.8 -> 0.00 mm
- net N$35: track 30.7 -> 0.00 mm, vias 4 -> 0
- net N$25: track 30.7 -> 0.00 mm, vias 2 -> 0
- net VSENSE_LEDG: track 29.4 -> 0.00 mm
- net N$34: track 27.1 -> 0.00 mm, vias 2 -> 0
- net GND: track 25.2 -> 0.00 mm
- net SWO: track 24.5 -> 0.00 mm
- net N$29: track 24.4 -> 0.00 mm, vias 1 -> 0
- net N$36: track 23.5 -> 0.00 mm
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- added copper zone on layer 16, net GND_MCU

Commit message: first attempt using modules
Parts:
- removed C10: 10uF, Eagle_Wurth_Elektronik_Passive_Capacitors_rev15a:2.6X1.6X1(BXCXA)
- removed C6, C7: 4.7uF, Eagle_Wurth_Elektronik_Passive_Capacitors_rev15a:WCAP-CSGP_0603_WAVE
- removed C8/1: (no value), Eagle_Wurth_Elektronik_Passive_Capacitors_rev15a:WCAP-CSGP_0603_WAVE
- removed D1, DZ1/1: MBR0540T1, mod_eagle_library_discrete_elements:SOD123
- removed D3: 1N4148WS, mod_eagle_library_discrete_elements:SOD323
- removed IC1/1: ILD4001, infineon:SC74_INFINEON
- removed L1: 1uH, EagleLibrary_Wuerth_Elektronik_eiSos_rev16a:WE-LQ_M
- removed L2/1: 68uH, EagleLibrary_Wuerth_Elektronik_eiSos_rev16a:WE-LQ_M
- removed R14/1: (no value), rcl:R0603
- removed U$4: LT1936, mod_eagle_library_pmic:MSOP8
- removed U1/1: PMXB56EN, mod_eagle_library_discrete_elements:DFN1010D-3
- added P1-1:C10: 10uF, Eagle_Wurth_Elektronik_Passive_Capacitors_rev15a:2.6X1.6X1(BXCXA)
- added P1-1:C2: 220pF, Eagle_Wurth_Elektronik_Passive_Capacitors_rev15a:WCAP-CSGP_0603_WAVE
- added P1-1:C3: 45uF, Eagle_Wurth_Elektronik_Passive_Capacitors_rev15a:2.6X1.6X1(BXCXA)
- added P1-1:C4, P1-1:C6, P1-1:C7: 4.7uF, Eagle_Wurth_Elektronik_Passive_Capacitors_rev15a:WCAP-CSGP_0603_WAVE
- added P1-1:D1, P2-1:DZ1: MBR0540T1, mod_eagle_library_discrete_elements:SOD123
- added P1-1:D3: 1N4148WS, mod_eagle_library_discrete_elements:SOD323
- added P1-1:L1: 1uH, EagleLibrary_Wuerth_Elektronik_eiSos_rev16a:WE-LQ_M
- added P1-1:R11: 10K, rcl:R0603
- added P1-1:R12: 17K5, rcl:R0603
- added P1-1:R13: 27K, rcl:R0603
- added P1-1:U$4: LT1936, mod_eagle_library_pmic:MSOP8
- added P2-1:C8/1: (no value), Eagle_Wurth_Elektronik_Passive_Capacitors_rev15a:WCAP-CSGP_0603_WAVE
- added P2-1:L2: 68uH, EagleLibrary_Wuerth_Elektronik_eiSos_rev16a:WE-LQ_M
- added P2-1:PMIC1: ILD4001, infineon:SC74_INFINEON
- added P2-1:R14: (no value), rcl:R0603
- added P2-1:U1: PMXB56EN, mod_eagle_library_discrete_elements:DFN1010D-3
- added R14, R15, R16: 100, rcl:R0603
- C2: value 220pF -> 4.7pF
- C3: value 45uF -> 4.7pF; device Eagle_Wurth_Elektronik_Passive_Capacitors_rev15a:2.6X1.6X1(BXCXA) -> Eagle_Wurth_Elektronik_Passive_Capacitors_rev15a:WCAP-CSGP_0603_WAVE
- C4: value 4.7uF -> 4.7pF
- R11: value 10K -> 22K
- R12: value 17K5 -> 22K
- R13: value 27K -> 22K
- moved R8 53.2 mm to (8.13, 5.33)
- moved R9 53.2 mm to (10.4, 5.33)
- moved R7 50.8 mm to (11.2, 8.13), turned to 0 degrees
- moved R10 47.1 mm to (11.2, 10.7), turned to 0 degrees
- moved C3 21.3 mm to (4.83, 49.8), flipped to the bottom
- moved R11 20.3 mm to (5.08, 52.1), flipped to the bottom, turned to 180 degrees
- moved D2 20.1 mm to (11.2, 31.5), flipped to the bottom
- moved R12 8.13 mm to (13.2, 48.5), flipped to the bottom, turned to 180 degrees
- moved C2 6.19 mm to (6.86, 54.1), flipped to the bottom
- moved C4 5.75 mm to (8.13, 48.0), flipped to the bottom
- moved R13 4.93 mm to (15.2, 46.5), flipped to the bottom
- renumbered U$7 to SW1
Connections:
- removed net DRIVER_LEDG/1: L2/1.1
- removed net ENABLE_LEDG/1: IC1/1.3
- removed net N$28: U$4.7, U$4.8
- removed net N$29: DZ1/1.A, L2/1.2, U1/1.3
- removed net N$30: C7.1, R13.1, U$4.5
- removed net N$33: C2.1, D3.C, U$4.1
- removed net N$34: C2.2, D1.C, L1.1, U$4.3
- removed net N$35: R11.2, R12.2, U$4.6
- removed net SUPPLY_3V3: C3.2, C4.1, D3.A, L1.2, R12.1
- removed net VSENSE_LEDG/1: IC1/1.6
- new net N$1: R11.1, R14.1, SW1.A
- new net N$10: R11.2, R12.2, R13.2
- new net N$11: C3.2, R15.1
- new net N$13: C2.2, R14.2
- new net N$16: R13.1, R16.2, SW1.E
- new net N$5: C2.1, C3.1, C4.1, SW1.C, SW1.D, SW1.GND1, SW1.GND2
- new net N$8: C4.2, R16.1
- new net P1-1:GND_MCU: P1-1:C10.1, P1-1:C3.1, P1-1:C4.2, P1-1:C6.2, P1-1:C7.2, P1-1:D1.A, P1-1:R11.1, P1-1:U$4.4, P1-1:U$4.9
- new net P1-1:N$28: P1-1:U$4.7, P1-1:U$4.8
- new net P1-1:N$30: P1-1:C7.1, P1-1:R13.1, P1-1:U$4.5
- new net P1-1:N$33: P1-1:C2.1, P1-1:D3.C, P1-1:U$4.1
- new net P1-1:N$34: P1-1:C2.2, P1-1:D1.C, P1-1:L1.1, P1-1:U$4.3
- new net P1-1:N$35: P1-1:R11.2, P1-1:R12.2, P1-1:U$4.6
- new net P1-1:SUPPLY_24V: P1-1:C10.2, P1-1:C6.1, P1-1:R13.2, P1-1:U$4.2
- new net P1-1:SUPPLY_3V3: P1-1:C3.2, P1-1:C4.1, P1-1:D3.A, P1-1:L1.2, P1-1:R12.1
- new net P2-1:ENABLE_LED: P2-1:PMIC1.3
- new net P2-1:N$2: P2-1:PMIC1.4, P2-1:R14.2, P2-1:U1.1
- new net P2-1:N$29: P2-1:DZ1.A, P2-1:L2.2, P2-1:U1.3
- net DRIVER_LEDG: now also P2-1:L2.1
- net GND_MCU: now also P2-1:C8/1.1, P2-1:PMIC1.2, P2-1:PMIC1.5, P2-1:R14.1, P2-1:U1.2; no longer C10.1, C3.1, C4.2, C6.2, C7.2, C8/1.1, D1.A, IC1/1.2, IC1/1.5, R11.1, R14/1.1, U$4.4, U$4.9, U1/1.2
- net N$2: now also R12.1, R15.2, SW1.B; no longer IC1/1.4, R14/1.2, U1/1.1
- net SUPPLY_24V: now also P2-1:C8/1.2, P2-1:DZ1.C, P2-1:PMIC1.1; no longer C10.2, C6.1, C8/1.2, DZ1/1.C, IC1/1.1, R13.2, U$4.2
- net VSENSE_LEDG: now also P2-1:PMIC1.6

Commit message: first layout of 4001
Parts:
- moved P2-1:R14 10.2 mm to (2.54, 28.7)
- moved P2-1:DZ1 6.43 mm to (9.40, 23.4)
- moved P2-1:U1 5.58 mm to (4.32, 26.2), turned to 0 degrees
- moved P2-1:C8/1 4.13 mm to (8.13, 29.5), turned to 180 degrees
- moved P2-1:L2 4.02 mm to (4.32, 22.1)
- moved D2 1.37 mm to (10.7, 32.8)
- moved P2-1:PMIC1 0.51 mm to (7.87, 26.7)
Routing:
- net SUPPLY_24V: track 0.00 -> 8.01 mm
- net P2-1:N$29: track 0.00 -> 5.37 mm
- net P2-1:N$2: track 0.00 -> 3.54 mm

Commit message: preliminary layout for LT1936
Parts:
- removed P1-1:C10: 10uF, Eagle_Wurth_Elektronik_Passive_Capacitors_rev15a:2.6X1.6X1(BXCXA)
- removed P1-1:C2: 220pF, Eagle_Wurth_Elektronik_Passive_Capacitors_rev15a:WCAP-CSGP_0603_WAVE
- removed P1-1:C3: 45uF, Eagle_Wurth_Elektronik_Passive_Capacitors_rev15a:2.6X1.6X1(BXCXA)
- removed P1-1:C4, P1-1:C6, P1-1:C7: 4.7uF, Eagle_Wurth_Elektronik_Passive_Capacitors_rev15a:WCAP-CSGP_0603_WAVE
- removed P1-1:D1, P2-1:DZ1: MBR0540T1, mod_eagle_library_discrete_elements:SOD123
- removed P1-1:D3: 1N4148WS, mod_eagle_library_discrete_elements:SOD323
- removed P1-1:L1: 1uH, EagleLibrary_Wuerth_Elektronik_eiSos_rev16a:WE-LQ_M
- removed P1-1:R11: 10K, rcl:R0603
- removed P1-1:R12: 17K5, rcl:R0603
- removed P1-1:R13: 27K, rcl:R0603
- removed P1-1:U$4: LT1936, mod_eagle_library_pmic:MSOP8
- removed P2-1:C8/1: (no value), Eagle_Wurth_Elektronik_Passive_Capacitors_rev15a:WCAP-CSGP_0603_WAVE
- removed P2-1:L2: 68uH, EagleLibrary_Wuerth_Elektronik_eiSos_rev16a:WE-LQ_M
- removed P2-1:PMIC1: ILD4001, infineon:SC74_INFINEON
- removed P2-1:R14: (no value), rcl:R0603
- removed P2-1:U1: PMXB56EN, mod_eagle_library_discrete_elements:DFN1010D-3
- added PMIC1:C10: 10uF, Eagle_Wurth_Elektronik_Passive_Capacitors_rev15a:2.6X1.6X1(BXCXA)
- added PMIC1:C2: 220pF, Eagle_Wurth_Elektronik_Passive_Capacitors_rev15a:WCAP-CSGP_0603_WAVE
- added PMIC1:C3: 45uF, Eagle_Wurth_Elektronik_Passive_Capacitors_rev15a:2.6X1.6X1(BXCXA)
- added PMIC1:C4, PMIC1:C6, PMIC1:C7: 4.7uF, Eagle_Wurth_Elektronik_Passive_Capacitors_rev15a:WCAP-CSGP_0603_WAVE
- added PMIC1:D1, PMIC2:DZ1, PMIC3:DZ1, PMIC4:DZ1, PMIC5:DZ1: MBR0540T1, mod_eagle_library_discrete_elements:SOD123
- added PMIC1:D3: 1N4148WS, mod_eagle_library_discrete_elements:SOD323
- added PMIC1:L1: 1uH, EagleLibrary_Wuerth_Elektronik_eiSos_rev16a:WE-LQ_M
- added PMIC1:R11: 10K, rcl:R0603
- added PMIC1:R12: 17K5, rcl:R0603
- added PMIC1:R13: 27K, rcl:R0603
- added PMIC1:U$4: LT1936, mod_eagle_library_pmic:MSOP8
- added PMIC2:C8, PMIC3:C8, PMIC4:C8, PMIC5:C8: (no value), Eagle_Wurth_Elektronik_Passive_Capacitors_rev15a:WCAP-CSGP_0603_WAVE
- added PMIC2:L2, PMIC3:L2, PMIC4:L2, PMIC5:L2: 68uH, EagleLibrary_Wuerth_Elektronik_eiSos_rev16a:WE-LQ_M
- added PMIC2:PMIC1, PMIC3:PMIC1, PMIC4:PMIC1, PMIC5:PMIC1: ILD4001, infineon:SC74_INFINEON
- added PMIC2:R14, PMIC3:R14, PMIC4:R14, PMIC5:R14: (no value), rcl:R0603
- added PMIC2:U1, PMIC3:U1, PMIC4:U1, PMIC5:U1: PMXB56EN, mod_eagle_library_discrete_elements:DFN1010D-3
- moved D2 55.2 mm to (57.3, 62.4)
- moved K1 54.2 mm to (28.4, 2.03), turned to 180 degrees
- moved R35 51.5 mm to (29.0, 6.10), turned to 90 degrees
- moved R36 51.3 mm to (25.4, 6.35), turned to 90 degrees
- moved R2 14.7 mm to (27.2, 38.4)
- moved SW1 13.5 mm to (9.40, 37.8)
- moved C5 13.2 mm to (29.5, 34.0)
- moved R3 9.94 mm to (30.7, 39.4)
- moved R15 5.89 mm to (7.37, 50.0)
- moved R13 4.79 mm to (11.2, 43.9)
- moved R12 2.84 mm to (10.7, 47.2)
- moved MCU1 2.03 mm to (18.3, 7.87)
Connections:
- removed net P1-1:GND_MCU: P1-1:C10.1, P1-1:C3.1, P1-1:C4.2, P1-1:C6.2, P1-1:C7.2, P1-1:D1.A, P1-1:R11.1, P1-1:U$4.4, P1-1:U$4.9
- removed net P1-1:N$28: P1-1:U$4.7, P1-1:U$4.8
- removed net P1-1:N$30: P1-1:C7.1, P1-1:R13.1, P1-1:U$4.5
- removed net P1-1:N$33: P1-1:C2.1, P1-1:D3.C, P1-1:U$4.1
- removed net P1-1:N$34: P1-1:C2.2, P1-1:D1.C, P1-1:L1.1, P1-1:U$4.3
- removed net P1-1:N$35: P1-1:R11.2, P1-1:R12.2, P1-1:U$4.6
- removed net P1-1:SUPPLY_24V: P1-1:C10.2, P1-1:C6.1, P1-1:R13.2, P1-1:U$4.2
- removed net P1-1:SUPPLY_3V3: P1-1:C3.2, P1-1:C4.1, P1-1:D3.A, P1-1:L1.2, P1-1:R12.1
- removed net P2-1:ENABLE_LED: P2-1:PMIC1.3
- removed net P2-1:N$2: P2-1:PMIC1.4, P2-1:R14.2, P2-1:U1.1
- removed net P2-1:N$29: P2-1:DZ1.A, P2-1:L2.2, P2-1:U1.3
- new net LEDB: MCU1.35, PMIC3:PMIC1.3
- new net LEDG: MCU1.36, PMIC2:PMIC1.3
- new net LEDR: MCU1.34, PMIC4:PMIC1.3
- new net LEDW: MCU1.33, PMIC5:PMIC1.3
- new net PMIC1:N$28: PMIC1:U$4.7, PMIC1:U$4.8
- new net PMIC1:N$30: PMIC1:C7.1, PMIC1:R13.1, PMIC1:U$4.5
- new net PMIC1:N$35: PMIC1:R11.2, PMIC1:R12.2, PMIC1:U$4.6
- new net PMIC1:PMIC_LT1936_BOOST: PMIC1:C2.1, PMIC1:D3.C, PMIC1:U$4.1
- new net PMIC1:PMIC_LT1936_SW: PMIC1:C2.2, PMIC1:D1.C, PMIC1:L1.1, PMIC1:U$4.3
- new net PMIC2:N$2: PMIC2:PMIC1.4, PMIC2:R14.2, PMIC2:U1.1
- new net PMIC2:N$29: PMIC2:DZ1.A, PMIC2:L2.2, PMIC2:U1.3
- new net PMIC3:N$2: PMIC3:PMIC1.4, PMIC3:R14.2, PMIC3:U1.1
- new net PMIC3:N$29: PMIC3:DZ1.A, PMIC3:L2.2, PMIC3:U1.3
- new net PMIC3:PMIC_IL4001_S24V: PMIC3:C8.2, PMIC3:DZ1.C, PMIC3:PMIC1.1
- new net PMIC4:N$2: PMIC4:PMIC1.4, PMIC4:R14.2, PMIC4:U1.1
- new net PMIC4:N$29: PMIC4:DZ1.A, PMIC4:L2.2, PMIC4:U1.3
- new net PMIC4:PMIC_IL4001_GND: PMIC4:C8.1, PMIC4:PMIC1.2, PMIC4:PMIC1.5, PMIC4:R14.1, PMIC4:U1.2
- new net PMIC5:N$2: PMIC5:PMIC1.4, PMIC5:R14.2, PMIC5:U1.1
- new net PMIC5:N$29: PMIC5:DZ1.A, PMIC5:L2.2, PMIC5:U1.3
- net DRIVER_LEDB: now also PMIC3:L2.1
- net DRIVER_LEDG: now also PMIC2:L2.1; no longer P2-1:L2.1
- net DRIVER_LEDR: now also PMIC4:L2.1
- net DRIVER_LEDW: now also PMIC5:L2.1
- net GND_MCU: now also PMIC1:C10.1, PMIC1:C3.1, PMIC1:C4.2, PMIC1:C6.2, PMIC1:C7.2, PMIC1:D1.A, PMIC1:R11.1, PMIC1:U$4.4, PMIC1:U$4.9, PMIC2:C8.1, PMIC2:PMIC1.2, PMIC2:PMIC1.5, PMIC2:R14.1, PMIC2:U1.2, PMIC3:C8.1, PMIC3:PMIC1.2, PMIC3:PMIC1.5, PMIC3:R14.1, PMIC3:U1.2, PMIC5:C8.1, PMIC5:PMIC1.2, PMIC5:PMIC1.5, PMIC5:R14.1, PMIC5:U1.2; no longer P2-1:C8/1.1, P2-1:PMIC1.2, P2-1:PMIC1.5, P2-1:R14.1, P2-1:U1.2
- net S3V3_MCU_VDD: now also PMIC1:C3.2, PMIC1:C4.1, PMIC1:D3.A, PMIC1:L1.2, PMIC1:R12.1
- net SUPPLY_24V: now also PMIC1:C10.2, PMIC1:C6.1, PMIC1:R13.2, PMIC1:U$4.2, PMIC2:C8.2, PMIC2:DZ1.C, PMIC2:PMIC1.1, PMIC4:C8.2, PMIC4:DZ1.C, PMIC4:PMIC1.1, PMIC5:C8.2, PMIC5:DZ1.C, PMIC5:PMIC1.1; no longer P2-1:C8/1.2, P2-1:DZ1.C, P2-1:PMIC1.1
- net VSENSE_LEDB: now also PMIC3:PMIC1.6
- net VSENSE_LEDG: now also PMIC2:PMIC1.6; no longer P2-1:PMIC1.6
- net VSENSE_LEDR: now also PMIC4:PMIC1.6
- net VSENSE_LEDW: now also PMIC5:PMIC1.6
Routing:
- net PMIC1:N$30: track 0.00 -> 19.4 mm
- net SUPPLY_24V: track 8.01 -> 0.00 mm
- net PMIC1:PMIC_LT1936_BOOST: track 0.00 -> 5.95 mm, vias 0 -> 2
- net P2-1:N$29: track 5.37 -> 0.00 mm
- net PMIC1:N$35: track 0.00 -> 4.16 mm
- net P2-1:N$2: track 3.54 -> 0.00 mm
- net GND_MCU: track 0.00 -> 1.31 mm, vias 0 -> 4
- added copper zone on layer 1, net GND_MCU
- added copper zone on layer 1, net PMIC1:PMIC_LT1936_BOOST
- added copper zone on layer 1, net PMIC1:PMIC_LT1936_SW
- added copper zone on layer 1, net S3V3_MCU_VDD
- added copper zone on layer 1, net SUPPLY_24V
Other:
- board size 39.6 x 59.4 mm -> 61.1 x 66.7 mm

Commit message: first layout for IL4001
Parts:
- moved PMIC2:U1 216.4 mm to (61.3, 26.8), turned to 90 degrees
- moved PMIC2:R14 214.4 mm to (61.0, 24.8)
- moved PMIC2:PMIC1 210.2 mm to (57.8, 27.9), turned to 270 degrees
- moved PMIC2:L2 207.8 mm to (65.5, 27.6), turned to 180 degrees
- moved PMIC2:DZ1 203.8 mm to (62.0, 30.9), turned to 270 degrees
- moved PMIC2:C8 198.0 mm to (56.9, 30.6), turned to 180 degrees
- moved PMIC1:R13 8.38 mm to (64.5, 61.3)
- moved PMIC1:C2 8.38 mm to (53.8, 66.0)
- moved D2 8.38 mm to (63.6, 67.8)
- moved PMIC1:C10 8.38 mm to (60.8, 61.7)
- moved PMIC1:C3 8.38 mm to (44.1, 61.7)
- moved PMIC1:C4 8.38 mm to (47.4, 61.2)
- moved PMIC1:C6 8.38 mm to (57.3, 61.2)
- moved PMIC1:C7 8.38 mm to (57.3, 58.2)
- moved PMIC1:L1 8.38 mm to (48.3, 67.1)
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Routing:
- net PMIC2:N$2: track 0.00 -> 5.43 mm
- added copper zone on layer 1, net PMIC2:N$29
Other:
- board size 61.1 x 66.7 mm -> 68.9 x 76.6 mm
