File: pro_event_light_a_mkI/pro_event_light_a_mkI_base_board.sch (EAGLE design)
At the start: 48 parts, among them K1 62201021121, SW1 ALPS_EC11D

Commit message: modelled all four IL4001 PMICs
Changed lines of the file:
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@@
 <pinref part="DZ1" gate="G$1" pin="C"/>
 <wire x1="170.18" y1="124.46" x2="170.18" y2="149.86" width="0.1524" layer="91"/>
-<label x="180.34" y="149.86" size="1.778" layer="95"/>
-<wire x1="170.18" y1="149.86" x2="208.28" y2="149.86" width="0.1524" layer="91"/>
 <wire x1="99.06" y1="149.86" x2="170.18" y2="149.86" width="0.1524" layer="91"/>
-<junction x="170.18" y="149.86"/>
 </segment>
 </net>
@@
 <moduleinsts>
 <moduleinst name="PMIC2" module="PMIC_IL4001" x="60.96" y="99.06"/>
-<moduleinst name="PMIC3" module="PMIC_IL4001" x="129.54" y="58.42"/>
 <moduleinst name="PMIC4" module="PMIC_IL4001" x="220.98" y="99.06"/>
-<moduleinst name="PMIC5" module="PMIC_IL4001" x="297.18" y="58.42"/>
+<moduleinst name="PMIC5" module="PMIC_IL4001" x="299.72" y="58.42"/>
+<moduleinst name="PMIC3" module="PMIC_IL4001" x="127" y="55.88"/>
 </moduleinsts>
 <instances>
@@
 <segment>
 <portref moduleinst="PMIC2" port="PMIC_IL4001_S24V"/>
-<wire x1="25.4" y1="104.14" x2="7.62" y2="104.14" width="0.1524" layer="91"/>
 <label x="7.62" y="104.14" size="1.778" layer="95"/>
-</segment>
-<segment>
-<wire x1="96.52" y1="63.5" x2="71.12" y2="63.5" width="0.1524" layer="91"/>
-<label x="73.66" y="63.5" size="1.778" layer="95"/>
+<wire x1="25.4" y1="104.14" x2="22.86" y2="104.14" width="0.1524" layer="91"/>
+<wire x1="22.86" y1="104.14" x2="7.62" y2="104.14" width="0.1524" layer="91"/>
+<wire x1="22.86" y1="104.14" x2="22.86" y2="63.5" width="0.1524" layer="91"/>
+<wire x1="22.86" y1="63.5" x2="91.44" y2="60.96" width="0.1524" layer="91"/>
+<junction x="22.86" y="104.14"/>
+<portref moduleinst="PMIC3" port="PMIC_IL4001_S24V"/>
+<wire x1="91.44" y1="60.96" x2="88.9" y2="63.5" width="0.1524" layer="91"/>
+<junction x="91.44" y="60.96"/>
 </segment>
 <segment>
 <portref moduleinst="PMIC5" port="PMIC_IL4001_S24V"/>
-<wire x1="261.62" y1="63.5" x2="236.22" y2="63.5" width="0.1524" layer="91"/>
+<wire x1="264.16" y1="63.5" x2="236.22" y2="63.5" width="0.1524" layer="91"/>
 <label x="238.76" y="63.5" size="1.778" layer="95"/>
 </segment>
@@
 <label x="172.72" y="134.62" size="1.778" layer="95" rot="R90"/>
 <wire x1="172.72" y1="152.4" x2="172.72" y2="63.5" width="0.1524" layer="91"/>
+<wire x1="172.72" y1="63.5" x2="162.56" y2="60.96" width="0.1524" layer="91"/>
 <portref moduleinst="PMIC3" port="PMIC_IL4001_KATHODE"/>
-<wire x1="172.72" y1="63.5" x2="165.1" y2="63.5" width="0.1524" layer="91"/>
 </segment>
 </net>
@@
 <junction x="172.72" y="210.82"/>
 <label x="149.86" y="210.82" size="1.778" layer="95"/>
-<portref moduleinst="PMIC3" port="PMIC_IL4001_VSENSE"/>
-<wire x1="165.1" y1="71.12" x2="167.64" y2="71.12" width="0.1524" layer="91"/>
 <wire x1="167.64" y1="71.12" x2="167.64" y2="139.7" width="0.1524" layer="91"/>
 <wire x1="167.64" y1="139.7" x2="139.7" y2="139.7" width="0.1524" layer="91"/>
 <wire x1="139.7" y1="139.7" x2="139.7" y2="210.82" width="0.1524" layer="91"/>
+<wire x1="167.64" y1="71.12" x2="162.56" y2="68.58" width="0.1524" layer="91"/>
+<portref moduleinst="PMIC3" port="PMIC_IL4001_VSENSE"/>
 </segment>
 </net>
@@
 <wire x1="347.98" y1="91.44" x2="347.98" y2="71.12" width="0.1524" layer="91"/>
 <portref moduleinst="PMIC5" port="PMIC_IL4001_VSENSE"/>
-<wire x1="347.98" y1="71.12" x2="332.74" y2="71.12" width="0.1524" layer="91"/>
+<wire x1="347.98" y1="71.12" x2="335.28" y2="71.12" width="0.1524" layer="91"/>
 </segment>
 </net>
@@
 <label x="317.5" y="134.62" size="1.778" layer="95" rot="R90"/>
 <portref moduleinst="PMIC5" port="PMIC_IL4001_KATHODE"/>
-<wire x1="332.74" y1="63.5" x2="340.36" y2="63.5" width="0.1524" layer="91"/>
+<wire x1="335.28" y1="63.5" x2="340.36" y2="63.5" width="0.1524" layer="91"/>
 <wire x1="340.36" y1="63.5" x2="340.36" y2="111.76" width="0.1524" layer="91"/>
 <wire x1="340.36" y1="111.76" x2="317.5" y2="111.76" width="0.1524" layer="91"/>
@@
 <segment>
 <portref moduleinst="PMIC2" port="PMIC_IL4001_GND"/>
-<wire x1="25.4" y1="81.28" x2="7.62" y2="81.28" width="0.1524" layer="91"/>
+<wire x1="25.4" y1="81.28" x2="15.24" y2="81.28" width="0.1524" layer="91"/>
 <label x="7.62" y="81.28" size="1.778" layer="95"/>
-</segment>
-<segment>
+<wire x1="15.24" y1="81.28" x2="7.62" y2="81.28" width="0.1524" layer="91"/>
+<wire x1="15.24" y1="81.28" x2="15.24" y2="40.64" width="0.1524" layer="91"/>
+<wire x1="15.24" y1="40.64" x2="91.44" y2="38.1" width="0.1524" layer="91"/>
+<junction x="15.24" y="81.28"/>
 <portref moduleinst="PMIC3" port="PMIC_IL4001_GND"/>
-<wire x1="93.98" y1="40.64" x2="71.12" y2="40.64" width="0.1524" layer="91"/>
-<label x="73.66" y="40.64" size="1.778" layer="95"/>
+<wire x1="91.44" y1="38.1" x2="88.9" y2="40.64" width="0.1524" layer="91"/>
+<junction x="91.44" y="38.1"/>
 </segment>
 <segment>
 <portref moduleinst="PMIC5" port="PMIC_IL4001_GND"/>
-<wire x1="261.62" y1="40.64" x2="236.22" y2="40.64" width="0.1524" layer="91"/>
+<wire x1="264.16" y1="40.64" x2="236.22" y2="40.64" width="0.1524" layer="91"/>
 <label x="241.3" y="40.64" size="1.778" layer="95"/>
 </segment>
 <segment>
-<wire x1="187.96" y1="81.28" x2="162.56" y2="81.28" width="0.1524" layer="91"/>
+<wire x1="185.42" y1="81.28" x2="162.56" y2="81.28" width="0.1524" layer="91"/>
 <label x="165.1" y="81.28" size="1.778" layer="95"/>
+<portref moduleinst="PMIC4" port="PMIC_IL4001_GND"/>
 </segment>
 </net>
@@
 <wire x1="60.96" y1="55.88" x2="63.5" y2="58.42" width="0.1524" layer="91"/>
 <portref moduleinst="PMIC3" port="PMIC_IL4001_EN_LED"/>
-<wire x1="63.5" y1="58.42" x2="93.98" y2="58.42" width="0.1524" layer="91"/>
+<wire x1="91.44" y1="55.88" x2="91.44" y2="58.42" width="0.1524" layer="91"/>
+<wire x1="91.44" y1="58.42" x2="63.5" y2="58.42" width="0.1524" layer="91"/>
 </segment>
 </net>
@@
 <wire x1="231.14" y1="55.88" x2="233.68" y2="58.42" width="0.1524" layer="91"/>
 <portref moduleinst="PMIC5" port="PMIC_IL4001_EN_LED"/>
-<wire x1="233.68" y1="58.42" x2="261.62" y2="58.42" width="0.1524" layer="91"/>
-</segment>
-</net>
+<wire x1="233.68" y1="58.42" x2="264.16" y2="58.42" width="0.1524" layer="91"/>
+</segment>
+</net>
